File: pcb/power.kicad_sch (KiCad schematic)
At the start: 17 parts

Commit message: Added guard ring
Optimized layout
Parts:
- removed D14: Blue, CRGM Passive:LED_0603_1608Metric, symbol Device:LED_Small
- removed JP8: ~, CRGM Connector:SolderJumper-2_P1.3mm_Bridged_RoundedPad1.0x1.5mm, symbol Jumper:SolderJumper_2_Bridged
- removed R9: 4.7K, CRGM Passive:R_0603_1608Metric, symbol Device:R_Small
- J10, J9, JP6, JP7, TP17, TP18, TP19: value ~ -> (none)
- R7: value 4.7K -> 10K; Digikey 541-3993-2-ND -> 541-3993-2-ND?; LCSC C2907166 -> C2907166?; MPN FRC0603J472 TS -> (none); Mouser 71-CRCW06034K70JNEAC -> 71-CRCW06034K70JNEAC?
- R8: value 1K -> 4.7K; Digikey 541-3991-2-ND -> 541-3993-2-ND; LCSC C2907113 -> C2907166; MN FOJAN -> FOJAN; MPN FRC0603J102 TS -> FRC0603J472 TS; Mouser 71-CRCW06031K00JNEAC -> 71-CRCW06034K70JNEAC
